File: PWR/PWR.sch (KiCad schematic (older format))
At the start: 22 parts

Commit message: Input added
Parts:
- added F?: Polyfuse, symbol Polyfuse
- added J?: Jack-DC, symbol Jack-DC
- added Q?: Q_PMOS_GDS, symbol Q_PMOS_GDS
Connections:
- net GND: now also J?.2, J?.3, Q?.1 (G)
- net VBUS: now also F?.2, J?.1
- net Vin_AfterSafety: now also Q?.3 (S)
- new net: F?.1, Q?.2 (D)
Other:
- moved on the sheet: 100u, 1k, 4k7, Q?, R?, SW?, U?

Commit message: Updates
Other:
- moved on the sheet: 100u, Q?, U?
Changed lines of the file:
@@
 L AP1117-33 U?
 U 1 1 5B706FF8
-P 6300 3300
-F 0 "U?" H 6150 3425 50  0000 C CNN
-F 1 "AP1117-33" H 6300 3425 50  0000 L CNN
-F 2 "TO_SOT_Packages_SMD:SOT-223-3Lead_TabPin2" H 6300 3500 50  0001 C CNN
-F 3 "" H 6400 3050 50  0001 C CNN
-	1    6300 3300
+P 6300 3150
+F 0 "U?" H 6150 3275 50  0000 C CNN
+F 1 "AP1117-33" H 6300 3275 50  0000 L CNN
+F 2 "TO_SOT_Packages_SMD:SOT-223-3Lead_TabPin2" H 6300 3350 50  0001 C CNN
+F 3 "" H 6400 2900 50  0001 C CNN
+	1    6300 3150
 	1    0    0    -1
 $EndComp
@@
 L GND #PWR?
 U 1 1 5B7072C9
-P 6300 3600
-F 0 "#PWR?" H 6300 3350 50  0001 C CNN
-F 1 "GND" H 6300 3450 50  0000 C CNN
-F 2 "" H 6300 3600 50  0001 C CNN
-F 3 "" H 6300 3600 50  0001 C CNN
-	1    6300 3600
+P 6300 3450
+F 0 "#PWR?" H 6300 3200 50  0001 C CNN
+F 1 "GND" H 6300 3300 50  0000 C CNN
+F 2 "" H 6300 3450 50  0001 C CNN
+F 3 "" H 6300 3450 50  0001 C CNN
+	1    6300 3450
 	1    0    0    -1
 $EndComp
@@
 Text GLabel 6000 4700 0    60   Input ~ 0
 Vin_AfterSafety
-Text GLabel 6000 3300 0    60   Input ~ 0
+Text GLabel 6000 3150 0    60   Input ~ 0
 Vin_AfterSafety
 Text GLabel 6000 6300 0    60   Input ~ 0
@@
 L CP 100u
 U 1 1 5B708149
-P 6800 3450
-F 0 "100u" H 6825 3550 50  0000 L CNN
-F 1 "CP" H 6825 3350 50  0000 L CNN
-F 2 "" H 6838 3300 50  0001 C CNN
-F 3 "" H 6800 3450 50  0001 C CNN
-	1    6800 3450
+P 6800 3300
+F 0 "100u" H 6825 3400 50  0000 L CNN
+F 1 "CP" H 6825 3200 50  0000 L CNN
+F 2 "" H 6838 3150 50  0001 C CNN
+F 3 "" H 6800 3300 50  0001 C CNN
+	1    6800 3300
 	1    0    0    -1
 $EndComp
@@
 L GND #PWR?
 U 1 1 5B708345
-P 6800 3600
-F 0 "#PWR?" H 6800 3350 50  0001 C CNN
-F 1 "GND" H 6800 3450 50  0000 C CNN
-F 2 "" H 6800 3600 50  0001 C CNN
-F 3 "" H 6800 3600 50  0001 C CNN
-	1    6800 3600
+P 6800 3450
+F 0 "#PWR?" H 6800 3200 50  0001 C CNN
+F 1 "GND" H 6800 3300 50  0000 C CNN
+F 2 "" H 6800 3450 50  0001 C CNN
+F 3 "" H 6800 3450 50  0001 C CNN
+	1    6800 3450
 	1    0    0    -1
 $EndComp
@@
 L Q_PMOS_GDS Q?
 U 1 1 5B70A66D
-P 7500 3400
-F 0 "Q?" H 7700 3450 50  0000 L CNN
-F 1 "Q_PMOS_GDS" H 7700 3350 50  0000 L CNN
-F 2 "" H 7700 3500 50  0001 C CNN
-F 3 "" H 7500 3400 50  0001 C CNN
-	1    7500 3400
+P 7500 3250
+F 0 "Q?" H 7700 3300 50  0000 L CNN
+F 1 "Q_PMOS_GDS" H 7700 3200 50  0000 L CNN
+F 2 "" H 7700 3350 50  0001 C CNN
+F 3 "" H 7500 3250 50  0001 C CNN
+	1    7500 3250
 	0    -1   -1   0
 $EndComp
@@
 	0    -1   -1   0
 $EndComp
-Text GLabel 8100 3300 2    60   Input ~ 0
+Text GLabel 8100 3150 2    60   Input ~ 0
 Vreg_3V3_HOT
 Text GLabel 8100 4700 2    60   Input ~ 0
@@
 	0    -1   -1   0
 $EndComp
-Text GLabel 7500 8400 3    60   Input ~ 0
-MosOn
-Text GLabel 11700 4400 0    60   Input ~ 0
-MosOn
-Text GLabel 7500 6600 3    60   Input ~ 0
-MosOn
-Text GLabel 7500 5000 3    60   Input ~ 0
-MosOn
-Text GLabel 7500 3600 3    60   Input ~ 0
-MosOn
 $Comp
 L Jack-DC J?
@@
 	6600 4700 7300 4700
 Wire Wire Line
-	6600 3300 7300 3300
+	6600 3150 7300 3150
 Wire Wire Line
 	7050 7050 7050 6800
@@
 Wire Wire Line
 	7050 8850 7050 8600
-Connection ~ 6800 3300
+Connection ~ 6800 3150
 Connection ~ 6800 4700
 Connection ~ 7050 6300
@@
 	8100 4700 7700 4700
 Wire Wire Line
-	7700 3300 8100 3300
+	7700 3150 8100 3150
 Wire Wire Line
 	14450 4950 14450 4900
@@
 	3000 5350 2850 5350
 Wire Notes Line
-	5150 4150 9150 4150
-Wire Notes Line
-	9150 4150 9150 5450
+	9150 4000 9150 5450
 Wire Notes Line
 	9150 5450 5150 5450
@@
 	4250 4700 4250 5900
 Wire Notes Line
-	5150 4050 9150 4050
-Wire Notes Line
-	9150 4050 9150 2650
-Wire Notes Line
-	9150 2650 5150 2650
-Wire Notes Line
-	5150 2650 5150 4050
+	5150 3900 9150 3900
+Wire Notes Line
+	9150 3900 9150 2500
+Wire Notes Line
+	9150 2500 5150 2500
+Wire Notes Line
+	5150 2500 5150 3900
 Wire Notes Line
 	9150 7350 9150 5550
@@
 Wire Notes Line
 	5150 5550 5150 5650
+Wire Notes Line
+	5150 4200 5150 4000
+Wire Notes Line
+	5150 4000 9150 4000
+Wire Wire Line
+	11250 4400 11700 4400
+Text Label 11250 4400 0    60   ~ 0
+MosOn
+Wire Wire Line
+	7500 8400 7500 8800
+Text Label 7500 8800 1    60   ~ 0
+MosOn
+Wire Wire Line
+	7500 6600 7500 6950
+Text Label 7500 6950 1    60   ~ 0
+MosOn
+Wire Wire Line
+	7500 5000 7500 5300
+Text Label 7500 5300 1    60   ~ 0
+MosOn
+Wire Wire Line
+	7500 3450 7500 3800
+Text Label 7500 3800 1    60   ~ 0
+MosOn
 $EndSCHEMATC
